File: FAN-plus40-SHIM.brd (EAGLE design)
At the start: 56 x 65 mm, 10 parts

Commit message: Connecting dots.
Routing:
- net VFAN: track 89.2 -> 90.3 mm
Other:
- board text added: "FAN-plus40-SHIM v1.0"
- board text removed: "FAN-plus-SHIM v1.0"
Changed lines of the file:
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@@
 <drawing>
 <settings>
-<setting alwaysvectorfont="yes"/>
+<setting alwaysvectorfont="no"/>
 <setting verticaltext="up"/>
 </settings>
@@
 <circle x="52.5" y="61.5" radius="3.2" width="0" layer="29"/>
 <circle x="52.5" y="61.5" radius="3.2" width="0" layer="30"/>
-<text x="9.197" y="2.571" size="1.27" layer="21" font="vector" ratio="24">FAN-plus-SHIM v1.0</text>
+<text x="8.181" y="2.571" size="1.27" layer="21" font="vector" ratio="24">FAN-plus40-SHIM v1.0</text>
 <text x="29.157" y="3.206" size="1.016" layer="21" font="vector" ratio="12">http://redscorp.net</text>
 <text x="29.157" y="1.936" size="1.016" layer="21" font="vector" ratio="12">(c) Andriy Golovnya</text>
@@
 <wire x1="43.18" y1="61.595" x2="42.291" y2="62.484" width="0.4064" layer="16"/>
 <wire x1="10.414" y1="59.309" x2="39.116" y2="59.309" width="0.4064" layer="1"/>
+<wire x1="43.18" y1="60.96" x2="44.2722" y2="60.96" width="0.1524" layer="16"/>
 </signal>
 <signal name="TACH">
@@
 <mfgpreviewcolor name="substratecolor" color="0xFF786E46"/>
 </mfgpreviewcolors>
+<errors>
+</errors>
 </board>
 </drawing>
