File: FAN-plus40-SHIM.sch (EAGLE design)
At the start: 8 parts

Commit message: Connecting dots.
Other:
- note added: "PI-FANP40S-0010"
- note removed: "PI-FANPS-0010"
Changed lines of the file:
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@@
 <plain>
 <text x="256.54" y="7.62" size="2.54" layer="94">1.0</text>
-<text x="198.12" y="7.62" size="2.54" layer="94">PI-FANPS-0010</text>
+<text x="198.12" y="7.62" size="2.54" layer="94">PI-FANP40S-0010</text>
 <text x="165.1" y="25.4" size="2.54" layer="94">Pi A+/B+ sized FAN-SHIM for Pi's 40-pin extension slot
 (c) Andriy Golovnya</text>
