File: FAN-zero30-SHIM.sch (EAGLE design)
At the start: 8 parts

Commit message: Connecting dots.
Other:
- note added: "PI-FANZ30S-0010"
- note removed: "PI-FANZS-0010"
Changed lines of the file:
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@@
 <plain>
 <text x="256.54" y="7.62" size="2.54" layer="94">1.0</text>
-<text x="198.12" y="7.62" size="2.54" layer="94">PI-FANZS-0010</text>
+<text x="198.12" y="7.62" size="2.54" layer="94">PI-FANZ30S-0010</text>
 <text x="165.1" y="25.4" size="2.54" layer="94">Pi Zero sized FAN-SHIM for Pi's 40-pin extension slot
 (c) Andriy Golovnya</text>
